File: pcb/Exoskeleton.kicad_pcb (KiCad board)
At the start: 4 copper layers, 114.2 x 134.5 mm, 55 parts, among them J11 PWR M5, J13 PWR M6, J15 TERM2, J16 BATT_SENSE, J17 DUMP_RESISTOR, J19 THERMAL_SW, J2 TERM, J3 PWR M1, J4 CANA, J5 PWR M2, J6 CANB, J7 PWR M3, J9 PWR M4, Q1 MMBT3906, Q2 IRFB4110, SW1 SW_SPDT, U1 Teensy4.1, U2 SN65HVD230, U3 TL431LP, U4 SN65HVD230

Commit message: Added mounting holes and removed excess CAN trace
Parts:
- added ?: , , F.Cu at (147.5, 94.5)
- added ?: , , F.Cu at (38.2, 46.2)
- added ?: , , F.Cu at (38.2, 175.2)
- added ?: , , F.Cu at (98.5, 175.0)
- added REF**: MountingHole_2.2mm_M2, MountingHole:MountingHole_2.2mm_M2, F.Cu at (146.2, 46.0)
Routing:
- net /CANH_B : track 30.4 -> 0.00 mm
